File: eagle_design/ext_tuner_rev1.sch (EAGLE design)
At the start: 209 parts, among them J1 SMA0.062, J2 SMA0.062, J3 AMPHENOL_A-1JB, J4 SMA0.062, J5 1734035-2, J6 AMPHENOL_A-1JB, U1 PG-103+, U11 74ALS04D, U2 HMC636ST89ETR, U3 HMC636ST89ETR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

Commit message: add ext tuner design
Parts:
- removed FAB6: 2118724, rf_shield_pn_2118724:RF_SHIELD_PN_2118724
- removed U$1: FULL-MINI-PCI-E, mini-pci-e:FULL-MINI-PCI-E
- removed X3: 679105700SMD, con-molex:679105700SMD
Changed lines of the file:
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@@
 <part name="SUPPLY132" library="supply2" deviceset="GND" device=""/>
 <part name="U4" library="pe4245" deviceset="PE4245" device="" value="4245-52"/>
-<part name="X3" library="con-molex" deviceset="679105700" device="SMD"/>
-<part name="U$1" library="mini-pci-e" deviceset="FULL-MINI-PCI-E" device=""/>
-<part name="FAB6" library="rf_shield_pn_2118724" deviceset="RF_SHIELD_PN_2118724" device="" value="2118724"/>
 </parts>
 <sheets>
@@
 <instance part="SUPPLY132" gate="GND" x="-355.6" y="142.24"/>
 <instance part="U4" gate="G$1" x="-10.16" y="35.56"/>
-<instance part="X3" gate="G$1" x="414.02" y="111.76"/>
-<instance part="U$1" gate="G$1" x="403.86" y="0"/>
-<instance part="U$1" gate="G$2" x="452.12" y="-5.08"/>
-<instance part="U$1" gate="G$3" x="459.74" y="-5.08"/>
-<instance part="FAB6" gate="G$1" x="406.4" y="182.88" smashed="yes">
-<attribute name="NAME" x="401.32" y="205.74" size="1.778" layer="95"/>
-<attribute name="VALUE" x="401.32" y="203.2" size="1.778" layer="96"/>
-</instance>
 </instances>
 <busses>
