File: eagle_design/SDR_at86rf215.brd (EAGLE design)
At the start: 167.6 x 78.7 mm, 221 parts, among them CON1 1734035-2, J1 SI-50170, J2 SJ-3523, J3 SMA0.062, J4 AMPHENOL_A-1JB, J5 5027740891, J6 AMPHENOL_A-1JB, J8 TC2030-CTX, Q1 MAR6-SM+, Q16 2N7002, SW1 45X45MM_TL3315, SW2 45X45MM_TL3315, SW3 45X45MM_TL3315, SW4 45X45MM_TL3315, SW5 45X45MM_TL3315, SW6 45X45MM_TL3315, SW7 45X45MM_TL3315, T1 0896FB15A0100, U1 AT86RF215, U10 NHD-C0216CZ-NSW-BBW-3V3, U11 MP34DT05TR-A, U12 ADP7156ARDZ-3.3-R7, U13 SN65LVDS1, U14 SN65LVDS1, U15 SN65LVDT2, U18 LAN8742, U2 ICE40HX8K-CT256, U3 TPS799X, U4 LD1117S12TR, U5 SN65LVDT2, U6 SN65LVDT2, U7 CS4344, U8 FT230XQ, U9 STM32H743ZIT6, X1 25MHz, X2 8MHZ, X3 ASVTX-12-A-40.000MHZ-H10-T

Commit message: update eagle files and schematic to reflect changes made to receiver when ext tuner was added
Parts:
- removed C31, C38: 100pF, m64library:C0603
- removed C34: 10nF, m64library:C0402
- removed C35: 33pF, m64library:C0402
- removed FLT2: HFCN-440D+, 195_est_library:MINICIRCUITS_FV1206
- removed L2, L3: 120nH, m64library:C0603
- removed Q1: MAR6-SM+, m64library:WW107
- removed R12: 82, resistor:R1206
Connections:
- removed net N$18: C34.2, C35.2, L3.2, R12.1
- removed net N$19: C38.1, FLT2.OUT
- removed net N$21: C28.2, FLT2.IN
- removed net N$3: C38.2, Q1.1
- removed net N$44: L2.2, R12.2
- removed net N$45: C31.1, L3.1, Q1.3
- net +5V: no longer L2.1
- net GND: no longer C34.1, C35.1, FLT2.3, FLT2.4, FLT2.5, FLT2.6, Q1.2, Q1.4
- net N$46: now also C28.2; no longer C31.2
Routing:
- net N$46: track 3.25 -> 16.1 mm
- net N$18: track 4.85 -> 0.00 mm
- net N$45: track 3.84 -> 0.00 mm
- net N$19: track 3.04 -> 0.00 mm
- net N$21: track 2.11 -> 0.00 mm
- net N$44: track 1.49 -> 0.00 mm
- net N$3: track 1.46 -> 0.00 mm
- net +5V: track 219.4 -> 218.6 mm
- net GND: track 328.3 -> 328.0 mm, vias 592 -> 581
